File: FioSaber/FioSaber Prototype.sch (EAGLE design)
At the start: 13 parts, among them CN1 1X4-BIG, P1 WIICHUCK

Commit message: vibraton motor
Parts:
- added C1: (no value), rcl:C-US025-025X050
- added D1: 1N4004, adafruit:1N4004
- added R5, R6: (no value), adafruit:R-US_0207/10
- added T1: 2N2222, adafruit:2N2222
- R1, R2, R3, R4: device rcl:R-US_0204/5 -> adafruit:R-US_0207/10
Connections:
- new net N$16: JP1.6, R6.2
- new net N$17: JP2.1, T1.E
- new net N$18: R6.1, T1.B
- new net N$19: C1.2, D1.A, T1.C
- new net N$2: JP2.3, R5.1
- new net N$20: C1.1, D1.C
Changed lines of the file:
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@@
 <part name="LED3" library="adafruit" deviceset="LED" device="3MM"/>
 <part name="LED4" library="adafruit" deviceset="LED" device="3MM"/>
-<part name="R1" library="rcl" deviceset="R-US_" device="0204/5"/>
-<part name="R2" library="rcl" deviceset="R-US_" device="0204/5"/>
-<part name="R3" library="rcl" deviceset="R-US_" device="0204/5"/>
-<part name="R4" library="rcl" deviceset="R-US_" device="0204/5"/>
+<part name="R1" library="adafruit" deviceset="R-US_" device="0207/10"/>
+<part name="R2" library="adafruit" deviceset="R-US_" device="0207/10"/>
+<part name="R3" library="adafruit" deviceset="R-US_" device="0207/10"/>
+<part name="R4" library="adafruit" deviceset="R-US_" device="0207/10"/>
 <part name="CN1" library="adafruit" deviceset="1X4" device="-BIG" value="1X4-BIG"/>
 <part name="P1" library="nintendo" deviceset="WIICHUCK" device=""/>
 <part name="U$1" library="headers(.1in)" deviceset="1X2" device=""/>
+<part name="T1" library="adafruit" deviceset="2N2222" device=""/>
+<part name="D1" library="adafruit" deviceset="1N4004" device=""/>
+<part name="C1" library="rcl" deviceset="C-US" device="025-025X050"/>
+<part name="R5" library="adafruit" deviceset="R-US_" device="0207/10"/>
+<part name="R6" library="adafruit" deviceset="R-US_" device="0207/10"/>
 </parts>
 <sheets>
@@
 <instance part="P1" gate="G$1" x="73.66" y="99.06" rot="R270"/>
 <instance part="U$1" gate="G$1" x="114.3" y="76.2"/>
+<instance part="T1" gate="G$1" x="195.58" y="71.12" rot="R90"/>
+<instance part="D1" gate="1" x="190.5" y="91.44" rot="R90"/>
+<instance part="C1" gate="G$1" x="180.34" y="91.44"/>
+<instance part="R5" gate="G$1" x="180.34" y="109.22"/>
+<instance part="R6" gate="G$1" x="195.58" y="60.96" rot="R270"/>
 </instances>
 <busses>
@@
 </segment>
 </net>
+<net name="N$2" class="0">
+<segment>
+<pinref part="JP2" gate="G$1" pin="3"/>
+<pinref part="R5" gate="G$1" pin="1"/>
+<wire x1="160.02" y1="101.6" x2="175.26" y2="101.6" width="0.1524" layer="91"/>
+<wire x1="175.26" y1="101.6" x2="175.26" y2="109.22" width="0.1524" layer="91"/>
+</segment>
+</net>
+<net name="N$16" class="0">
+<segment>
+<pinref part="JP1" gate="G$1" pin="6"/>
+<wire x1="106.68" y1="93.98" x2="109.22" y2="93.98" width="0.1524" layer="91"/>
+<wire x1="109.22" y1="93.98" x2="109.22" y2="55.88" width="0.1524" layer="91"/>
+<wire x1="109.22" y1="55.88" x2="195.58" y2="55.88" width="0.1524" layer="91"/>
+<pinref part="R6" gate="G$1" pin="2"/>
+</segment>
+</net>
+<net name="N$17" class="0">
+<segment>
+<pinref part="JP2" gate="G$1" pin="1"/>
+<wire x1="160.02" y1="106.68" x2="160.02" y2="114.3" width="0.1524" layer="91"/>
+<pinref part="T1" gate="G$1" pin="E"/>
+<wire x1="160.02" y1="114.3" x2="200.66" y2="114.3" width="0.1524" layer="91"/>
+<wire x1="200.66" y1="114.3" x2="200.66" y2="73.66" width="0.1524" layer="91"/>
+</segment>
+</net>
+<net name="N$18" class="0">
+<segment>
+<pinref part="R6" gate="G$1" pin="1"/>
+<pinref part="T1" gate="G$1" pin="B"/>
+<wire x1="195.58" y1="66.04" x2="195.58" y2="68.58" width="0.1524" layer="91"/>
+</segment>
+</net>
+<net name="N$19" class="0">
+<segment>
+<pinref part="T1" gate="G$1" pin="C"/>
+<pinref part="D1" gate="1" pin="A"/>
+<wire x1="190.5" y1="73.66" x2="190.5" y2="83.82" width="0.1524" layer="91"/>
+<wire x1="190.5" y1="88.9" x2="190.5" y2="83.82" width="0.1524" layer="91"/>
+<pinref part="C1" gate="G$1" pin="2"/>
+<wire x1="190.5" y1="83.82" x2="180.34" y2="83.82" width="0.1524" layer="91"/>
+<wire x1="180.34" y1="83.82" x2="180.34" y2="86.36" width="0.1524" layer="91"/>
+</segment>
+</net>
+<net name="N$20" class="0">
+<segment>
+<pinref part="D1" gate="1" pin="C"/>
+<wire x1="190.5" y1="93.98" x2="190.5" y2="101.6" width="0.1524" layer="91"/>
+<wire x1="190.5" y1="101.6" x2="180.34" y2="101.6" width="0.1524" layer="91"/>
+<pinref part="C1" gate="G$1" pin="1"/>
+<wire x1="180.34" y1="101.6" x2="180.34" y2="93.98" width="0.1524" layer="91"/>
+</segment>
+</net>

Commit message: added fiosaber gerbers
Parts:
- added U$2: 1X2, headers(.1in):1X2
- renumbered CN1 to I2C, JP1 to FIOL, JP2 to FIOR
Connections:
- net N$19: now also U$2.1
- net N$20: now also R5.2, U$2.2
Changed lines of the file:
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@@
 <parts>
 <part name="FRAME1" library="SparkFun" deviceset="FRAME-LETTER" device=""/>
-<part name="JP1" library="SparkFun" deviceset="M14" device=""/>
-<part name="JP2" library="SparkFun" deviceset="M14" device=""/>
+<part name="FIOL" library="SparkFun" deviceset="M14" device=""/>
+<part name="FIOR" library="SparkFun" deviceset="M14" device=""/>
 <part name="LED1" library="adafruit" deviceset="LED" device="3MM"/>
 <part name="LED2" library="adafruit" deviceset="LED" device="3MM"/>
@@
 <part name="R3" library="adafruit" deviceset="R-US_" device="0207/10"/>
 <part name="R4" library="adafruit" deviceset="R-US_" device="0207/10"/>
-<part name="CN1" library="adafruit" deviceset="1X4" device="-BIG" value="1X4-BIG"/>
+<part name="I2C" library="adafruit" deviceset="1X4" device="-BIG" value="1X4-BIG"/>
 <part name="P1" library="nintendo" deviceset="WIICHUCK" device=""/>
 <part name="U$1" library="headers(.1in)" deviceset="1X2" device=""/>
@@
 <part name="R5" library="adafruit" deviceset="R-US_" device="0207/10"/>
 <part name="R6" library="adafruit" deviceset="R-US_" device="0207/10"/>
+<part name="U$2" library="headers(.1in)" deviceset="1X2" device=""/>
 </parts>
 <sheets>
@@
 <instance part="FRAME1" gate="G$1" x="0" y="0"/>
 <instance part="FRAME1" gate="G$2" x="147.32" y="0"/>
-<instance part="JP1" gate="G$1" x="96.52" y="88.9" rot="MR180"/>
-<instance part="JP2" gate="G$1" x="170.18" y="88.9" rot="R180"/>
+<instance part="FIOL" gate="G$1" x="96.52" y="88.9" rot="MR180"/>
+<instance part="FIOR" gate="G$1" x="170.18" y="88.9" rot="R180"/>
 <instance part="LED1" gate="G$1" x="119.38" y="137.16"/>
 <instance part="LED2" gate="G$1" x="132.08" y="137.16"/>
@@
 <instance part="R3" gate="G$1" x="144.78" y="124.46"/>
 <instance part="R4" gate="G$1" x="157.48" y="124.46"/>
-<instance part="CN1" gate="G$1" x="124.46" y="88.9"/>
+<instance part="I2C" gate="G$1" x="124.46" y="88.9"/>
 <instance part="P1" gate="G$1" x="73.66" y="99.06" rot="R270"/>
 <instance part="U$1" gate="G$1" x="114.3" y="76.2"/>
@@
 <instance part="R5" gate="G$1" x="180.34" y="109.22"/>
 <instance part="R6" gate="G$1" x="195.58" y="60.96" rot="R270"/>
+<instance part="U$2" gate="G$1" x="203.2" y="91.44" rot="R270"/>
 </instances>
 <busses>
@@
 <wire x1="114.3" y1="142.24" x2="71.12" y2="142.24" width="0.1524" layer="91"/>
 <wire x1="71.12" y1="142.24" x2="71.12" y2="104.14" width="0.1524" layer="91"/>
-<pinref part="JP1" gate="G$1" pin="2"/>
+<pinref part="FIOL" gate="G$1" pin="2"/>
 <wire x1="106.68" y1="104.14" x2="71.12" y2="104.14" width="0.1524" layer="91"/>
 <pinref part="P1" gate="G$1" pin="GND"/>
@@
 <wire x1="106.68" y1="104.14" x2="116.84" y2="104.14" width="0.1524" layer="91"/>
 <wire x1="116.84" y1="104.14" x2="116.84" y2="91.44" width="0.1524" layer="91"/>
-<pinref part="CN1" gate="G$1" pin="1"/>
+<pinref part="I2C" gate="G$1" pin="1"/>
 <wire x1="116.84" y1="91.44" x2="119.38" y2="91.44" width="0.1524" layer="91"/>
 </segment>
@@
 <net name="N$5" class="0">
 <segment>
-<pinref part="JP2" gate="G$1" pin="12"/>
+<pinref part="FIOR" gate="G$1" pin="12"/>
 <wire x1="160.02" y1="78.74" x2="134.62" y2="78.74" width="0.1524" layer="91"/>
 <wire x1="134.62" y1="78.74" x2="134.62" y2="109.22" width="0.1524" layer="91"/>
@@
 <net name="N$6" class="0">
 <segment>
-<pinref part="JP2" gate="G$1" pin="11"/>
+<pinref part="FIOR" gate="G$1" pin="11"/>
 <wire x1="160.02" y1="81.28" x2="137.16" y2="81.28" width="0.1524" layer="91"/>
 <wire x1="137.16" y1="81.28" x2="137.16" y2="111.76" width="0.1524" layer="91"/>
@@
 <net name="N$7" class="0">
 <segment>
-<pinref part="JP2" gate="G$1" pin="10"/>
+<pinref part="FIOR" gate="G$1" pin="10"/>
 <wire x1="160.02" y1="83.82" x2="139.7" y2="83.82" width="0.1524" layer="91"/>
 <pinref part="R3" gate="G$1" pin="1"/>
@@
 <net name="N$8" class="0">
 <segment>
-<pinref part="JP2" gate="G$1" pin="9"/>
+<pinref part="FIOR" gate="G$1" pin="9"/>
 <wire x1="160.02" y1="86.36" x2="152.4" y2="86.36" width="0.1524" layer="91"/>
 <pinref part="R4" gate="G$1" pin="1"/>
@@
 <net name="N$1" class="0">
 <segment>
-<pinref part="JP1" gate="G$1" pin="1"/>
+<pinref part="FIOL" gate="G$1" pin="1"/>
 <wire x1="106.68" y1="106.68" x2="88.9" y2="106.68" width="0.1524" layer="91"/>
 <wire x1="88.9" y1="106.68" x2="88.9" y2="68.58" width="0.1524" layer="91"/>
@@
 <wire x1="106.68" y1="106.68" x2="132.08" y2="106.68" width="0.1524" layer="91"/>
 <wire x1="132.08" y1="106.68" x2="132.08" y2="88.9" width="0.1524" layer="91"/>
-<pinref part="CN1" gate="G$1" pin="2"/>
+<pinref part="I2C" gate="G$1" pin="2"/>
 <wire x1="132.08" y1="88.9" x2="119.38" y2="88.9" width="0.1524" layer="91"/>
 </segment>
@@
 <net name="N$3" class="0">
 <segment>
-<pinref part="JP1" gate="G$1" pin="3"/>
+<pinref part="FIOL" gate="G$1" pin="3"/>
 <wire x1="106.68" y1="101.6" x2="91.44" y2="101.6" width="0.1524" layer="91"/>
 <wire x1="91.44" y1="101.6" x2="91.44" y2="66.04" width="0.1524" layer="91"/>
@@
 <wire x1="106.68" y1="101.6" x2="114.3" y2="101.6" width="0.1524" layer="91"/>
 <wire x1="114.3" y1="101.6" x2="114.3" y2="86.36" width="0.1524" layer="91"/>
-<pinref part="CN1" gate="G$1" pin="3"/>
+<pinref part="I2C" gate="G$1" pin="3"/>
 <wire x1="114.3" y1="86.36" x2="119.38" y2="86.36" width="0.1524" layer="91"/>
 </segment>
@@
 <net name="N$4" class="0">
 <segment>
-<pinref part="JP1" gate="G$1" pin="4"/>
+<pinref part="FIOL" gate="G$1" pin="4"/>
 <wire x1="106.68" y1="99.06" x2="93.98" y2="99.06" width="0.1524" layer="91"/>
 <wire x1="93.98" y1="99.06" x2="93.98" y2="63.5" width="0.1524" layer="91"/>
@@
 <wire x1="106.68" y1="99.06" x2="111.76" y2="99.06" width="0.1524" layer="91"/>
 <wire x1="111.76" y1="99.06" x2="111.76" y2="83.82" width="0.1524" layer="91"/>
-<pinref part="CN1" gate="G$1" pin="4"/>
+<pinref part="I2C" gate="G$1" pin="4"/>
 <wire x1="111.76" y1="83.82" x2="119.38" y2="83.82" width="0.1524" layer="91"/>
 </segment>
@@
 <net name="N$14" class="0">
 <segment>
-<pinref part="JP2" gate="G$1" pin="4"/>
+<pinref part="FIOR" gate="G$1" pin="4"/>
 <wire x1="160.02" y1="99.06" x2="175.26" y2="99.06" width="0.1524" layer="91"/>
 <wire x1="175.26" y1="99.06" x2="175.26" y2="63.5" width="0.1524" layer="91"/>
@@
 <net name="N$15" class="0">
 <segment>
-<pinref part="JP2" gate="G$1" pin="5"/>
+<pinref part="FIOR" gate="G$1" pin="5"/>
 <wire x1="160.02" y1="96.52" x2="172.72" y2="96.52" width="0.1524" layer="91"/>
 <wire x1="172.72" y1="96.52" x2="172.72" y2="66.04" width="0.1524" layer="91"/>
@@
 <net name="N$2" class="0">
 <segment>
-<pinref part="JP2" gate="G$1" pin="3"/>
+<pinref part="FIOR" gate="G$1" pin="3"/>
 <pinref part="R5" gate="G$1" pin="1"/>
 <wire x1="160.02" y1="101.6" x2="175.26" y2="101.6" width="0.1524" layer="91"/>
@@
 <net name="N$16" class="0">
 <segment>
-<pinref part="JP1" gate="G$1" pin="6"/>
+<pinref part="FIOL" gate="G$1" pin="6"/>
 <wire x1="106.68" y1="93.98" x2="109.22" y2="93.98" width="0.1524" layer="91"/>
 <wire x1="109.22" y1="93.98" x2="109.22" y2="55.88" width="0.1524" layer="91"/>
@@
 <net name="N$17" class="0">
 <segment>
-<pinref part="JP2" gate="G$1" pin="1"/>
+<pinref part="FIOR" gate="G$1" pin="1"/>
 <wire x1="160.02" y1="106.68" x2="160.02" y2="114.3" width="0.1524" layer="91"/>
 <pinref part="T1" gate="G$1" pin="E"/>
-<wire x1="160.02" y1="114.3" x2="200.66" y2="114.3" width="0.1524" layer="91"/>
-<wire x1="200.66" y1="114.3" x2="200.66" y2="73.66" width="0.1524" layer="91"/>
+<wire x1="160.02" y1="114.3" x2="223.52" y2="114.3" width="0.1524" layer="91"/>
+<wire x1="223.52" y1="114.3" x2="223.52" y2="73.66" width="0.1524" layer="91"/>
+<wire x1="223.52" y1="73.66" x2="200.66" y2="73.66" width="0.1524" layer="91"/>
 </segment>
 </net>
@@
 <wire x1="190.5" y1="83.82" x2="180.34" y2="83.82" width="0.1524" layer="91"/>
 <wire x1="180.34" y1="83.82" x2="180.34" y2="86.36" width="0.1524" layer="91"/>
+<wire x1="190.5" y1="83.82" x2="203.2" y2="83.82" width="0.1524" layer="91"/>
+<pinref part="U$2" gate="G$1" pin="1"/>
+<wire x1="203.2" y1="83.82" x2="203.2" y2="88.9" width="0.1524" layer="91"/>
 </segment>
 </net>
@@
 <pinref part="C1" gate="G$1" pin="1"/>
 <wire x1="180.34" y1="101.6" x2="180.34" y2="93.98" width="0.1524" layer="91"/>
-</segment>
-</net>
+<wire x1="190.5" y1="101.6" x2="200.66" y2="101.6" width="0.1524" layer="91"/>
+<pinref part="U$2" gate="G$1" pin="2"/>
+<wire x1="200.66" y1="101.6" x2="200.66" y2="88.9" width="0.1524" layer="91"/>
+<pinref part="R5" gate="G$1" pin="2"/>
+<wire x1="185.42" y1="109.22" x2="220.98" y2="109.22" width="0.1524" layer="91"/>
+<wire x1="220.98" y1="109.22" x2="220.98" y2="101.6" width="0.1524" layer="91"/>
+<wire x1="220.98" y1="101.6" x2="200.66" y2="101.6" width="0.1524" layer="91"/>
+</segment>
+</net>
