File: FioSaber/FioSaber Prototype.brd (EAGLE design)
At the start: 25.4 x 44.1 mm, 13 parts, among them CN1 1X4-BIG, P1 WIICHUCK

Commit message: vibraton motor
Parts:
- added C1: (no value), rcl:C025-025X050
- added D1: 1N4004, adafruit:DO41-10
- added R5, R6: (no value), adafruit:0207/10
- added T1: 2N2222, adafruit:TO92-EBC-OVAL
- R1, R2, R3, R4: device rcl:0204/5 -> adafruit:0207/10
- moved U$1 36.1 mm to (23.5, 5.08)
- moved R4 12.3 mm to (13.3, 34.3), turned to 90 degrees
- moved R3 9.09 mm to (10.8, 34.3), turned to 90 degrees
- moved R2 6.38 mm to (8.26, 34.3), turned to 90 degrees
- moved R1 4.96 mm to (5.71, 34.3), turned to 90 degrees
- moved LED4 3.86 mm to (18.4, 26.7)
- moved LED3 3.24 mm to (18.4, 31.1)
- moved LED2 2.62 mm to (18.4, 35.6)
- moved LED1 2.01 mm to (18.4, 40.0)
- moved JP1 1.27 mm to (1.27, 44.5)
- moved JP2 1.27 mm to (24.1, 44.5)
- moved CN1 1.27 mm to (12.7, 17.8)
Connections:
- new net N$16: JP1.6, R6.2
- new net N$17: JP2.1, T1.E
- new net N$18: R6.1, T1.B
- new net N$19: C1.2, D1.A, T1.C
- new net N$2: JP2.3, R5.1
- new net N$20: C1.1, D1.C
Routing:
- net N$2: track 0.00 -> 40.9 mm, vias 0 -> 4
- net N$19: track 0.00 -> 40.1 mm, vias 0 -> 4
- net N$20: track 0.00 -> 36.7 mm, vias 0 -> 2
- net N$3: track 45.8 -> 9.20 mm, vias 4 -> 2
- net N$17: track 0.00 -> 34.2 mm, vias 0 -> 4
- net N$14: track 18.3 -> 46.8 mm, vias 0 -> 6
- net N$15: track 21.5 -> 35.6 mm
- net N$21: track 0.00 -> 12.1 mm
- net N$18: track 0.00 -> 12.1 mm, vias 0 -> 1
- net N$12: track 5.08 -> 16.3 mm, vias 0 -> 2
- net N$16: track 0.00 -> 11.2 mm, vias 0 -> 1
- net N$11: track 7.62 -> 14.6 mm
- net N$5: track 33.2 -> 36.8 mm, vias 2 -> 4
- net N$23: track 0.00 -> 3.30 mm
- net N$8: track 18.8 -> 15.9 mm, vias 0 -> 2
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Other:
- board size 25.4 x 44.1 mm -> 25.4 x 45.3 mm
- board text added: "A"
- board text added: "B"
- board text added: "C"
- board text added: "D"
- board text added: "R5"
- board text added: "R6"
- board text removed: "L1"
- board text removed: "L2"
- board text removed: "L3"
- board text removed: "L4"

Commit message: added fiosaber gerbers
Parts:
- removed CN1: 1X4-BIG, adafruit:1X04-BIG
- added I2C: 1X4-BIG, adafruit:1X04-BIG
- added U$2: 1X2, headers(.1in):1X2
- moved D1 0.64 mm to (19.1, 17.8)
- moved T1 0.63 mm to (11.4, 23.5)
- renumbered JP1 to FIOL, JP2 to FIOR
Connections:
- net N$1: now also I2C.2; no longer CN1.2
- net N$13: now also I2C.1; no longer CN1.1
- net N$19: now also U$2.1
- net N$20: now also R5.2, U$2.2
- net N$3: now also I2C.3; no longer CN1.3
- net N$4: now also I2C.4; no longer CN1.4
Routing:
- net N$3: track 9.20 -> 48.4 mm, vias 2 -> 6
- net N$1: track 50.7 -> 72.4 mm, vias 9 -> 4
- net N$21: track 12.1 -> 0.00 mm
- net N$2: track 40.9 -> 29.4 mm, vias 4 -> 1
- net N$5: track 36.8 -> 32.4 mm, vias 4 -> 1
- net N$23: track 3.30 -> 0.00 mm
- net N$20: track 36.7 -> 33.5 mm, vias 2 -> 3
- net N$14: track 46.8 -> 49.0 mm
- net N$17: track 34.2 -> 35.5 mm, vias 4 -> 2
- net N$22: track 1.09 -> 0.00 mm
- net N$4: track 43.2 -> 42.2 mm, vias 4 -> 2
- net N$18: track 12.1 -> 11.4 mm
- net N$6: track 25.4 -> 25.0 mm, vias 1 -> 2
- net N$16: track 11.2 -> 11.3 mm, vias 1 -> 2
- net N$19: track 40.1 -> 40.2 mm, vias 4 -> 3
Other:
- board text added: "VIBRATE"

Commit message: schematic tweaks
Parts:
- C1: value (none) -> 0.1µF
- R1, R2, R3, R4, R6: value (none) -> 1kΩ
- R5: value (none) -> 33Ω
Changed lines of the file:
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@@
 <element name="LED3" library="adafruit" package="LED3MM" value="" x="18.415" y="31.115"/>
 <element name="LED4" library="adafruit" package="LED3MM" value="" x="18.415" y="26.67"/>
-<element name="R1" library="adafruit" package="0207/10" value="" x="5.715" y="34.29" rot="R90"/>
-<element name="R2" library="adafruit" package="0207/10" value="" x="8.255" y="34.29" rot="R90"/>
-<element name="R3" library="adafruit" package="0207/10" value="" x="10.795" y="34.29" rot="R90"/>
-<element name="R4" library="adafruit" package="0207/10" value="" x="13.335" y="34.29" rot="R90"/>
+<element name="R1" library="adafruit" package="0207/10" value="1kΩ" x="5.715" y="34.29" rot="R90"/>
+<element name="R2" library="adafruit" package="0207/10" value="1kΩ" x="8.255" y="34.29" rot="R90"/>
+<element name="R3" library="adafruit" package="0207/10" value="1kΩ" x="10.795" y="34.29" rot="R90"/>
+<element name="R4" library="adafruit" package="0207/10" value="1kΩ" x="13.335" y="34.29" rot="R90"/>
 <element name="I2C" library="adafruit" package="1X04-BIG" value="1X4-BIG" x="12.7" y="18.0975" rot="R270"/>
 <element name="P1" library="nintendo" package="MEMOREX_RECEIVER" value="WIICHUCK" x="12.7" y="0"/>
@@
 <element name="T1" library="adafruit" package="TO92-EBC-OVAL" value="2N2222" x="11.43" y="23.495" rot="R90"/>
 <element name="D1" library="adafruit" package="DO41-10" value="1N4004" x="19.05" y="17.78" rot="R90"/>
-<element name="C1" library="rcl" package="C025-025X050" value="" x="1.905" y="3.81" rot="R90"/>
-<element name="R5" library="adafruit" package="0207/10" value="" x="5.715" y="21.59" rot="R270"/>
-<element name="R6" library="adafruit" package="0207/10" value="" x="8.255" y="21.59" rot="R90"/>
+<element name="C1" library="rcl" package="C025-025X050" value="0.1µF" x="1.905" y="3.81" rot="R90"/>
+<element name="R5" library="adafruit" package="0207/10" value="33Ω" x="5.715" y="21.59" rot="R270"/>
+<element name="R6" library="adafruit" package="0207/10" value="1kΩ" x="8.255" y="21.59" rot="R90"/>
 <element name="U$2" library="headers(.1in)" package="1X2" value="1X2" x="6.985" y="10.4775"/>
 </elements>

Commit message: prototype b
Parts:
- R1, R2, R3, R4: value 1kΩ -> 100Ω
Changed lines of the file:
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@@
 <element name="LED3" library="adafruit" package="LED3MM" value="" x="18.415" y="31.115"/>
 <element name="LED4" library="adafruit" package="LED3MM" value="" x="18.415" y="26.67"/>
-<element name="R1" library="adafruit" package="0207/10" value="1kΩ" x="5.715" y="34.29" rot="R90"/>
-<element name="R2" library="adafruit" package="0207/10" value="1kΩ" x="8.255" y="34.29" rot="R90"/>
-<element name="R3" library="adafruit" package="0207/10" value="1kΩ" x="10.795" y="34.29" rot="R90"/>
-<element name="R4" library="adafruit" package="0207/10" value="1kΩ" x="13.335" y="34.29" rot="R90"/>
+<element name="R1" library="adafruit" package="0207/10" value="100Ω" x="5.715" y="34.29" rot="R90"/>
+<element name="R2" library="adafruit" package="0207/10" value="100Ω" x="8.255" y="34.29" rot="R90"/>
+<element name="R3" library="adafruit" package="0207/10" value="100Ω" x="10.795" y="34.29" rot="R90"/>
+<element name="R4" library="adafruit" package="0207/10" value="100Ω" x="13.335" y="34.29" rot="R90"/>
 <element name="I2C" library="adafruit" package="1X04-BIG" value="1X4-BIG" x="12.7" y="18.0975" rot="R270"/>
 <element name="P1" library="nintendo" package="MEMOREX_RECEIVER" value="WIICHUCK" x="12.7" y="0"/>
