File: FioSaber/FioSaber.sch (EAGLE design)
At the start: 18 parts, among them P1 WIICHUCK, T1 2N2222

Commit message: board tweaks
Parts:
- IN, OUT: device adafruit:JST_2PIN-SMT-RA -> adafruit:JST_2PIN-THM-RA
Changed lines of the file:
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@@
 <part name="D1" library="adafruit" deviceset="1N4004" device=""/>
 <part name="S1" library="adafruit" deviceset="EG1218" device="S"/>
-<part name="IN" library="adafruit" deviceset="JST_2PIN" device="-SMT-RA"/>
-<part name="OUT" library="adafruit" deviceset="JST_2PIN" device="-SMT-RA"/>
+<part name="IN" library="adafruit" deviceset="JST_2PIN" device="-THM-RA"/>
+<part name="OUT" library="adafruit" deviceset="JST_2PIN" device="-THM-RA"/>
 <part name="D2" library="adafruit" deviceset="1N4004" device=""/>
 <part name="R2" library="adafruit" deviceset="R-US_" device="0207/7" value="100Ω"/>
