File: FioSaber/FioSaber.brd (EAGLE design)
At the start: 26.7 x 55.5 mm, 18 parts, among them P1 WIICHUCK, T1 2N2222

Commit message: board tweaks
Parts:
- IN, OUT: device adafruit:JST-PH-2-SMT-RA -> adafruit:JST-PH-2-THM-RA
- moved IN 5.08 mm to (3.81, 48.9), flipped to the top
- moved OUT 5.08 mm to (21.6, 48.9), flipped to the top
- moved MOTOR 1.27 mm to (11.4, 50.2)
- moved T1 1.27 mm to (22.9, 5.71), flipped to the top
- moved C1 1.27 mm to (12.7, 53.3), flipped to the top, turned to 180 degrees
- moved S1 0.64 mm to (12.7, 34.9)
- moved SWITCH 0.64 mm to (12.7, 28.6)
- moved R1 0.63 mm to (7.94, 42.5), flipped to the top, turned to 270 degrees
- moved R2 0.63 mm to (11.1, 42.5), flipped to the top
- moved R3 0.63 mm to (14.3, 42.5), flipped to the top, turned to 270 degrees
- moved R4 0.63 mm to (17.5, 42.5), flipped to the top
- moved D1 0.32 mm to (7.30, 18.4), flipped to the top
- moved D2 0.32 mm to (18.1, 18.4), flipped to the top
- flipped MODE to the top
- flipped TX to the top
Routing:
- net N$13: track 61.9 -> 50.9 mm, vias 5 -> 4
- net N$16: track 28.5 -> 20.0 mm
- net N$1: track 50.5 -> 57.2 mm, vias 4 -> 6
- net N$18: track 44.2 -> 50.3 mm, vias 4 -> 2
- net N$6: track 15.5 -> 11.0 mm
- net N$8: track 11.9 -> 16.1 mm
- net N$20: track 52.9 -> 48.9 mm
- net N$11: track 23.0 -> 19.0 mm
- net N$9: track 72.1 -> 68.4 mm, vias 7 -> 3
- net N$17: track 45.0 -> 41.7 mm, vias 3 -> 2
- net N$25: track 42.1 -> 39.1 mm, vias 4 -> 3
- net N$2: track 46.2 -> 43.4 mm, vias 3 -> 2
- net N$7: track 13.5 -> 11.2 mm
- net N$4: track 40.1 -> 38.8 mm
- net N$5: track 20.2 -> 19.3 mm
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Other:
- board size 26.7 x 55.5 mm -> 28.6 x 53.6 mm

Commit message: back to square board
Parts:
- moved T1 0.32 mm to (22.5, 5.71)
Routing:
- net N$19: track 60.8 -> 55.9 mm
- net N$17: track 41.7 -> 42.8 mm, vias 2 -> 3
- net N$18: track 50.3 -> 49.7 mm, vias 2 -> 3
- net N$20: track 48.9 -> 48.3 mm
Other:
- board size 28.6 x 53.6 mm -> 26.7 x 53.6 mm
